File: boards/Balloon/Balloon.sch (EAGLE design)
At the start: 23 parts

Commit message: Balloon board updated with new power boards and library components
Other:
- moved on the sheet: R1, R2

Commit message: Ballon v4 as submitted to manufacturing
Parts:
- added SERV0: (no value), SparkFun-Connectors:M03PTH
- ARDUINO: value ARDUINO_PRO_MINI -> ARDUINO_PRO_MINI-NOSILK; device OpenSpace:ARDUINO_PRO_MINI -> OpenSpace:ARDUINO_PRO_MINI-NOSILK
- GPS: value VENUS_GPS -> VENUS_GPS-NOSILK; device OpenSpace:VENUS_GPS -> OpenSpace:VENUS_GPS-NOSILK
- MAIN, RADIO: device OpenSpace:POWER-TPS6300X -> OpenSpace:POWER-TPS6300X-NOSILK
- R1: value (none) -> 1.2K
- R2: value (none) -> 3.9K
- THERM0: device SparkFun-Connectors:M02JST-PTH-2 -> SparkFun-Passives:RESISTOR0805-RES
Connections:
- new net D11: ARDUINO.D11*, SERV0.3
- net 3.3V: now also SERV0.2
- net GND: now also SERV0.1
Other:
- moved on the sheet: GPS, R_T0, R_T1, R_T2, THERM1, THERM2
