File: boards/Balloon/Balloon.brd (EAGLE design)
At the start: 41.9 x 69.8 mm, 23 parts

Commit message: Balloon board updated with new power boards and library components
Routing:
- net GND: track 127.2 -> 0.00 mm
- net 3.3V: track 59.9 -> 0.00 mm
- net 1.8V: track 40.0 -> 0.00 mm
- net 5V: track 28.4 -> 0.00 mm

Commit message: Ballon v4 as submitted to manufacturing
Parts:
- added SERV0: (no value), SparkFun-Connectors:1X03
- ARDUINO: value ARDUINO_PRO_MINI -> ARDUINO_PRO_MINI-NOSILK; device OpenSpace:ARDUINO_PRO_MINI -> OpenSpace:ARDUINO_PRO_MINI-NOSILK
- GPS: value VENUS_GPS -> VENUS_GPS-NOSILK; device OpenSpace:VENUS_GPS -> OpenSpace:VENUS_GPS-NOSILK
- MAIN, RADIO: device OpenSpace:POWER-TPS6300X -> OpenSpace:POWER-TPS6300X-NOSILK
- R1: value (none) -> 1.2K
- R2: value (none) -> 3.9K
- THERM0: device SparkFun-Connectors:JST-2-PTH -> SparkFun-Passives:0805
- moved R2 60.3 mm to (59.7, 26.7), turned to 90 degrees
- moved R1 55.7 mm to (59.7, 30.5), turned to 90 degrees
- moved GPS 53.4 mm to (53.3, 9.53), turned to 270 degrees
- moved ARDUINO 45.4 mm to (48.3, 28.6), turned to 270 degrees
- moved R_T2 43.2 mm to (49.5, 27.9), turned to 270 degrees
- moved R_SCL 41.4 mm to (24.1, 19.1)
- moved SHIFT_FROM_RADIO 41.0 mm to (19.7, 14.0), turned to 180 degrees
- moved R_T1 39.6 mm to (47.0, 27.9), turned to 270 degrees
- moved MAIN 39.1 mm to (5.08, 32.4), turned to 270 degrees
- moved SHIFT_TO_RADIO 38.9 mm to (23.5, 14.0), turned to 0 degrees
- moved R_SDA 37.6 mm to (19.1, 19.1)
- moved R_T0 36.1 mm to (44.5, 27.9), turned to 270 degrees
- moved I2C_1 33.1 mm to (33.0, 3.81), turned to 0 degrees
- moved I2C_0 27.4 mm to (33.0, 11.4), turned to 0 degrees
- moved XTEND 27.0 mm to (23.5, 5.08), turned to 180 degrees
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Connections:
- new net D11: ARDUINO.D11*, SERV0.3
- net 3.3V: now also SERV0.2
- net GND: now also SERV0.1
Routing:
- net GND: track 0.00 -> 220.4 mm, vias 0 -> 1
- net 3.3V: track 0.00 -> 128.9 mm
- net SDA: track 0.00 -> 96.1 mm
- net SCL: track 0.00 -> 95.0 mm
- net 1.8V: track 0.00 -> 94.2 mm
- net 5V: track 0.00 -> 47.2 mm, vias 0 -> 1
- net D4: track 0.00 -> 40.8 mm, vias 0 -> 1
- net A2: track 0.00 -> 38.4 mm
- net A1: track 0.00 -> 36.2 mm
- net RX: track 0.00 -> 32.4 mm
- net D5: track 0.00 -> 31.4 mm, vias 0 -> 1
- net N$1: track 0.00 -> 16.2 mm, vias 0 -> 1
- net N$2: track 0.00 -> 14.2 mm
- net A0: track 0.00 -> 12.2 mm, vias 0 -> 1
- net D11: track 0.00 -> 10.4 mm, vias 0 -> 1
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Other:
- board size 41.9 x 69.8 mm -> 63.5 x 38.1 mm
- board text added: "Balloon v4"
- board text removed: "425-922-9404"
- board text removed: "CXXI SAT v4"

Commit message: Minor position changes on the Balloon board
Parts:
- moved MAIN 1.27 mm to (5.08, 33.7)
Routing:
- net GND: track 220.4 -> 221.7 mm
- net 3.3V: track 128.9 -> 130.2 mm
- net 1.8V: track 94.2 -> 94.9 mm
Other:
- board text added: "Balloon v5"
Changed lines of the file:
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@@
 <hole x="13.97" y="34.29" drill="3.2"/>
 <hole x="13.97" y="3.81" drill="3.2"/>
-<text x="62.23" y="31.75" size="2.54" layer="22" ratio="12" rot="MR0">Balloon v4</text>
+<text x="62.23" y="31.75" size="2.54" layer="22" ratio="12" rot="MR0">Balloon v5</text>
 <text x="10.795" y="7.62" size="2.54" layer="21" ratio="12" rot="R90">Balloon v4</text>
 </plain>
@@
 <element name="SHIFT_FROM_RADIO" library="OpenSpace" package="SC70" value="SN74LVC1T45-DCK" x="19.685" y="13.97" smashed="yes" rot="R180"/>
 <element name="SHIFT_TO_RADIO" library="OpenSpace" package="SC70" value="SN74LVC1T45-DCK" x="23.495" y="13.97" smashed="yes"/>
-<element name="MAIN" library="OpenSpace" package="POWER-TPS6300X-NOSILK" value="3.3V" x="5.08" y="32.385" rot="R270"/>
+<element name="MAIN" library="OpenSpace" package="POWER-TPS6300X-NOSILK" value="3.3V" x="5.08" y="33.655" rot="R270"/>
 <element name="RADIO" library="OpenSpace" package="POWER-TPS6300X-NOSILK" value="5V" x="5.08" y="4.445" rot="R90"/>
 <element name="THERM0" library="SparkFun-Passives" package="0805" value="10K" x="39.37" y="17.145" rot="R180"/>
@@
 <wire x1="6.35" y1="16.51" x2="6.35" y2="17.145" width="1.016" layer="16"/>
 <wire x1="6.35" y1="17.145" x2="3.81" y2="19.685" width="1.016" layer="16"/>
-<wire x1="3.81" y1="19.685" x2="3.81" y2="22.225" width="1.016" layer="16"/>
-<wire x1="3.81" y1="22.225" x2="3.81" y2="34.925" width="1.016" layer="16"/>
+<wire x1="3.81" y1="19.685" x2="3.81" y2="23.495" width="1.016" layer="16"/>
+<wire x1="3.81" y1="23.495" x2="3.81" y2="36.195" width="1.016" layer="16"/>
 <wire x1="21.495" y1="5.08" x2="21.495" y2="3.715" width="0.6096" layer="16"/>
 <wire x1="21.495" y1="3.715" x2="19.05" y2="1.27" width="0.6096" layer="16"/>
@@
 <contactref element="THERM0" pad="2"/>
 <contactref element="SERV0" pad="2"/>
-<wire x1="6.35" y1="22.225" x2="6.35" y2="20.32" width="0.254" layer="1"/>
+<wire x1="6.35" y1="23.495" x2="6.35" y2="20.32" width="0.254" layer="1"/>
 <wire x1="6.35" y1="20.32" x2="12.7" y2="13.97" width="0.254" layer="1"/>
 <wire x1="12.7" y1="11.43" x2="12.7" y2="13.97" width="0.254" layer="1"/>
@@
 <wire x1="1.27" y1="6.35" x2="1.27" y2="27.94" width="1.016" layer="1"/>
 <wire x1="1.27" y1="27.94" x2="6.35" y2="33.02" width="1.016" layer="1"/>
-<wire x1="6.35" y1="33.02" x2="6.35" y2="34.925" width="1.016" layer="1"/>
+<wire x1="6.35" y1="33.02" x2="6.35" y2="36.195" width="1.016" layer="1"/>
 <wire x1="59.69" y1="31.38" x2="56.78" y2="34.29" width="0.254" layer="1"/>
 <wire x1="56.78" y1="34.29" x2="53.975" y2="34.29" width="0.254" layer="1"/>
@@
 <wire x1="53.34" y1="34.925" x2="53.34" y2="36.83" width="0.254" layer="1"/>
 <wire x1="53.34" y1="36.83" x2="52.705" y2="37.465" width="0.254" layer="1"/>
-<wire x1="52.705" y1="37.465" x2="8.89" y2="37.465" width="0.254" layer="1"/>
-<wire x1="8.89" y1="37.465" x2="6.35" y2="34.925" width="0.254" layer="1"/>
+<wire x1="52.705" y1="37.465" x2="7.62" y2="37.465" width="0.254" layer="1"/>
+<wire x1="7.62" y1="37.465" x2="6.35" y2="36.195" width="0.254" layer="1"/>
 </signal>
 <signal name="5V">
