File: boards/Jonah/Jonah.sch (EAGLE design)
At the start: 10 parts

Commit message: First pass at Jonah board v2
Parts:
- removed XBEE: XBEE-1B2, SparkFun-RF:XBEE-1B2
- added RF_TX: 434 MHz, SparkFun-Connectors:M04PTH
Connections:
- removed net N$3: ARDUINO.TXO, XBEE.DIN
- removed net N$4: ARDUINO.RXI, XBEE.DOUT
- net 3.3V: now also RF_TX.3; no longer XBEE.VDD
- net GND: now also RF_TX.1; no longer XBEE.GND
- net N$1: now also ARDUINO.TXO, RF_TX.2; no longer ARDUINO.RST0, XBEE.RESET
Changed lines of the file:
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@@
 <part name="MAIN" library="OpenSpace" deviceset="POWER" device="-TPS6300X-NOSILK" value="3.3V"/>
 <part name="THERM0" library="SparkFun-Passives" deviceset="RESISTOR" device="0805-RES" value="10K"/>
-<part name="XBEE" library="SparkFun-RF" deviceset="XBEE-1" device="B2"/>
 <part name="P+5" library="SparkFun-Aesthetics" deviceset="3.3V" device=""/>
 <part name="GND3" library="SparkFun-Aesthetics" deviceset="GND" device=""/>
+<part name="RF_TX" library="SparkFun-Connectors" deviceset="M04" device="PTH" value="434 MHz"/>
 </parts>
 <sheets>
@@
 <instance part="MAIN" gate="POWER" x="35.56" y="33.02"/>
 <instance part="THERM0" gate="G$1" x="111.76" y="40.64" rot="R90"/>
-<instance part="XBEE" gate="G$1" x="5.08" y="-35.56"/>
-<instance part="P+5" gate="G$1" x="-17.78" y="-7.62"/>
-<instance part="GND3" gate="1" x="-17.78" y="-68.58"/>
+<instance part="P+5" gate="G$1" x="10.16" y="-12.7"/>
+<instance part="GND3" gate="1" x="10.16" y="-40.64"/>
+<instance part="RF_TX" gate="G$1" x="2.54" y="-27.94"/>
 </instances>
 <busses>
@@
 </segment>
 <segment>
-<pinref part="XBEE" gate="G$1" pin="GND"/>
-<wire x1="-15.24" y1="-48.26" x2="-17.78" y2="-48.26" width="0.1524" layer="91"/>
-<wire x1="-17.78" y1="-48.26" x2="-17.78" y2="-66.04" width="0.1524" layer="91"/>
+<pinref part="RF_TX" gate="G$1" pin="1"/>
 <pinref part="GND3" gate="1" pin="GND"/>
+<wire x1="7.62" y1="-30.48" x2="10.16" y2="-30.48" width="0.1524" layer="91"/>
+<wire x1="10.16" y1="-30.48" x2="10.16" y2="-38.1" width="0.1524" layer="91"/>
 </segment>
 </net>
@@
 </segment>
 <segment>
-<pinref part="XBEE" gate="G$1" pin="VDD"/>
+<pinref part="RF_TX" gate="G$1" pin="3"/>
 <pinref part="P+5" gate="G$1" pin="3.3V"/>
-<wire x1="-15.24" y1="-25.4" x2="-17.78" y2="-25.4" width="0.1524" layer="91"/>
-<wire x1="-17.78" y1="-25.4" x2="-17.78" y2="-7.62" width="0.1524" layer="91"/>
+<wire x1="7.62" y1="-25.4" x2="10.16" y2="-25.4" width="0.1524" layer="91"/>
+<wire x1="10.16" y1="-25.4" x2="10.16" y2="-12.7" width="0.1524" layer="91"/>
 </segment>
 </net>
@@
 <net name="N$1" class="0">
 <segment>
-<pinref part="ARDUINO" gate="G$1" pin="RST0"/>
-<wire x1="86.36" y1="-30.48" x2="91.44" y2="-30.48" width="0.1524" layer="91"/>
-<wire x1="91.44" y1="-30.48" x2="91.44" y2="-10.16" width="0.1524" layer="91"/>
-<wire x1="91.44" y1="-10.16" x2="-25.4" y2="-10.16" width="0.1524" layer="91"/>
-<wire x1="-25.4" y1="-10.16" x2="-25.4" y2="-35.56" width="0.1524" layer="91"/>
-<pinref part="XBEE" gate="G$1" pin="RESET"/>
-<wire x1="-25.4" y1="-35.56" x2="-15.24" y2="-35.56" width="0.1524" layer="91"/>
-</segment>
-</net>
-<net name="N$3" class="0">
-<segment>
+<pinref part="RF_TX" gate="G$1" pin="2"/>
+<wire x1="7.62" y1="-27.94" x2="25.4" y2="-27.94" width="0.1524" layer="91"/>
+<wire x1="25.4" y1="-27.94" x2="25.4" y2="-22.86" width="0.1524" layer="91"/>
 <pinref part="ARDUINO" gate="G$1" pin="TXO"/>
-<wire x1="50.8" y1="-22.86" x2="48.26" y2="-22.86" width="0.1524" layer="91"/>
-<wire x1="48.26" y1="-22.86" x2="48.26" y2="-12.7" width="0.1524" layer="91"/>
-<wire x1="48.26" y1="-12.7" x2="-22.86" y2="-12.7" width="0.1524" layer="91"/>
-<wire x1="-22.86" y1="-12.7" x2="-22.86" y2="-30.48" width="0.1524" layer="91"/>
-<pinref part="XBEE" gate="G$1" pin="DIN"/>
-<wire x1="-22.86" y1="-30.48" x2="-15.24" y2="-30.48" width="0.1524" layer="91"/>
-</segment>
-</net>
-<net name="N$4" class="0">
-<segment>
-<pinref part="ARDUINO" gate="G$1" pin="RXI"/>
-<wire x1="50.8" y1="-25.4" x2="45.72" y2="-25.4" width="0.1524" layer="91"/>
-<wire x1="45.72" y1="-25.4" x2="45.72" y2="-15.24" width="0.1524" layer="91"/>
-<wire x1="45.72" y1="-15.24" x2="-20.32" y2="-15.24" width="0.1524" layer="91"/>
-<wire x1="-20.32" y1="-15.24" x2="-20.32" y2="-27.94" width="0.1524" layer="91"/>
-<pinref part="XBEE" gate="G$1" pin="DOUT"/>
-<wire x1="-20.32" y1="-27.94" x2="-15.24" y2="-27.94" width="0.1524" layer="91"/>
-</segment>
-</net>
+<wire x1="25.4" y1="-22.86" x2="50.8" y2="-22.86" width="0.1524" layer="91"/>
+</segment>
+</net>

Commit message: Jonah board v2
Rearranged things, and now use SparkFun's KLP radio, not an Xbee.

Also, made some space and holes for attaching to a rod.
Parts:
- ARDUINO: value ARDUINO_PRO_MINI -> ARDUINO_PRO_MINI-NOSILK; device OpenSpace:ARDUINO_PRO_MINI -> OpenSpace:ARDUINO_PRO_MINI-NOSILK
Changed lines of the file:
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@@
 <parts>
 <part name="BMP085" library="SparkFun" deviceset="M06" device="SIP"/>
-<part name="ARDUINO" library="OpenSpace" deviceset="ARDUINO_PRO_MINI" device=""/>
+<part name="ARDUINO" library="OpenSpace" deviceset="ARDUINO_PRO_MINI" device="-NOSILK"/>
 <part name="P+1" library="SparkFun-Aesthetics" deviceset="3.3V" device=""/>
 <part name="P+2" library="SparkFun-Aesthetics" deviceset="3.3V" device=""/>
