File: boards/Power/TPS6300x/TPS6300x.brd (EAGLE design)
At the start: 26.7 x 10.2 mm, 12 parts

Commit message: Removed voltage divider on power board
Vina wasn't the place to do a voltage divider, and I realized that I
really didn't need one -- I don't want a cutoff for the Lithium primary
batteries, and the Li-Ion batteries have a built-in low-voltage cutoff.
Parts:
- removed R1: 53.6k, SparkFun-Passives:0805
- removed R2: 100k, SparkFun-Passives:0805
- removed UVLO: 1.7/2.6, SparkFun-Passives:SJ_3
- moved EN_SEL 1.91 mm to (11.4, 1.27)
Connections:
- removed net N$4: R1.1, R2.2, UVLO.3
- removed net VINA: TPS63001.8, UVLO.2
- net 1.8V: now also TPS63001.8; no longer R1.2, UVLO.1
- net GND: no longer R2.1
Routing:
- net N$4: track 13.0 -> 0.00 mm
- net 1.8V: track 45.5 -> 33.5 mm
- net VINA: track 7.39 -> 0.00 mm
- net GND: track 31.9 -> 30.0 mm, vias 4 -> 3
Other:
- board text added: "v4"
- board text removed: "v3"
