File: boards/APRS/APRS.brd (EAGLE design)
At the start: 50.8 x 38.1 mm, 19 parts

Commit message: Added Jonah receiver to APRS v3
Parts:
- added JONAH_RECEIVER: RADIO-KLP-RECEIVER-NOSILK, OpenSpace:RADIO-KLP-RECEIVER-NOSILK
- moved RADIOMETRIX_HX1 2.54 mm to (29.2, 33.0)
- moved ARDUINO 2.54 mm to (34.3, 15.2)
- moved LEVEL_SHIFT 2.54 mm to (44.5, 15.2)
- moved SDA_PU 2.54 mm to (7.62, 15.2)
- moved I2C_0 2.54 mm to (12.7, 7.62)
- moved POWER3 2.54 mm to (11.4, 7.62)
- moved POWER5 2.54 mm to (22.9, 7.62)
- moved GPS0 2.54 mm to (39.4, 12.7)
- moved I2C_TRANS 2.54 mm to (20.3, 12.7)
- moved J$1 2.54 mm to (2.54, 24.1)
- moved LED1 2.54 mm to (48.9, 25.4)
- moved R1 2.54 mm to (45.1, 25.4)
- moved R_T0 2.54 mm to (30.5, 17.1)
- moved R_T1 2.54 mm to (33.0, 17.1)
- moved R_T2 2.54 mm to (35.6, 17.1)
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Connections:
- new net JONAH_RX: ARDUINO.D11*, JONAH_RECEIVER.2
- net 5V: now also JONAH_RECEIVER.4, JONAH_RECEIVER.5
- net GND: now also JONAH_RECEIVER.1, JONAH_RECEIVER.6, JONAH_RECEIVER.7
Routing:
- net 5V: track 128.3 -> 162.7 mm
- net GND: track 113.1 -> 134.2 mm
- net JONAH_RX: track 0.00 -> 16.3 mm
- net A2: track 40.4 -> 41.5 mm
Other:
- board size 50.8 x 38.1 mm -> 50.8 x 40.6 mm
- board text added: "APRS v3"
- board text removed: "APRS v2"

Commit message: Fixed misnamed I2C pull-ups
Parts:
- moved SCL_PU 2.54 mm to (7.62, 15.2)
- moved SDA_PU 2.54 mm to (7.62, 12.7)
Connections:
- net SCL: now also SCL_PU.1; no longer SDA_PU.1
- net SDA: now also SDA_PU.1; no longer SCL_PU.1
Changed lines of the file:
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@@
 </element>
 <element name="I2C_TRANS" library="OpenSpace" package="SO8" value="PCA9306-D" x="20.32" y="12.7" rot="R270"/>
-<element name="SCL_PU" library="SparkFun-Passives" package="0805" value="3.3k" x="7.62" y="12.7" rot="R180"/>
-<element name="SDA_PU" library="SparkFun-Passives" package="0805" value="3.3k" x="7.62" y="15.24" rot="R180"/>
+<element name="SDA_PU" library="SparkFun-Passives" package="0805" value="3.3k" x="7.62" y="12.7" rot="R180"/>
+<element name="SCL_PU" library="SparkFun-Passives" package="0805" value="3.3k" x="7.62" y="15.24" rot="R180"/>
 <element name="I2C_0" library="SparkFun-Connectors" package="1X04" value="" x="12.7" y="7.62" rot="R90"/>
 <element name="JONAH_RECEIVER" library="OpenSpace" package="RADIO-KLP-RECEIVER-NOSILK" value="RADIO-KLP-RECEIVER-NOSILK" x="28.575" y="1.905" smashed="yes">
@@
 <contactref element="POWER3" pad="VCC+"/>
 <contactref element="I2C_TRANS" pad="2"/>
+<contactref element="SDA_PU" pad="2"/>
 <contactref element="SCL_PU" pad="2"/>
-<contactref element="SDA_PU" pad="2"/>
 <contactref element="I2C_0" pad="2"/>
 <wire x1="12.7" y1="10.16" x2="11.43" y2="11.43" width="0.254" layer="16"/>
@@
 <signal name="SCL">
 <contactref element="I2C_TRANS" pad="3"/>
-<contactref element="SDA_PU" pad="1"/>
+<contactref element="SCL_PU" pad="1"/>
 <contactref element="I2C_0" pad="4"/>
 <wire x1="8.52" y1="15.24" x2="12.7" y2="15.24" width="0.254" layer="1"/>
@@
 <signal name="SDA">
 <contactref element="I2C_TRANS" pad="4"/>
-<contactref element="SCL_PU" pad="1"/>
+<contactref element="SDA_PU" pad="1"/>
 <contactref element="I2C_0" pad="3"/>
 <wire x1="8.52" y1="12.7" x2="12.7" y2="12.7" width="0.254" layer="1"/>

Commit message: APRS v4 -- Added RX_EN
I couldn't solder the Arduino board directly because the level
shifter was breaking uploading sketches, so I added an RX_EN
jumper.
Parts:
- added RX_EN: (no value), SparkFun-Passives:1X02
- moved LED1 19.7 mm to (29.2, 25.4)
- moved R1 19.7 mm to (25.4, 25.4)
Connections:
- new net N$7: LEVEL_SHIFT.3, RX_EN.2
- net RX: now also RX_EN.1; no longer LEVEL_SHIFT.3
Routing:
- net N$7: track 0.00 -> 20.7 mm, vias 0 -> 1
- net D4: track 20.2 -> 5.60 mm
- net RX: track 12.2 -> 2.54 mm, vias 1 -> 0
- net GND: track 134.2 -> 139.4 mm
Other:
- board text added: "APRS v4"
- board text removed: "APRS v3"
Changed lines of the file:
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@@
 <wire x1="50.8" y1="40.64" x2="0" y2="40.64" width="0" layer="20"/>
 <wire x1="0" y1="40.64" x2="0" y2="0" width="0" layer="20"/>
-<text x="49.53" y="36.83" size="2.54" layer="22" font="vector" ratio="15" rot="MR0">APRS v3</text>
+<text x="49.53" y="36.83" size="2.54" layer="22" font="vector" ratio="15" rot="MR0">APRS v4</text>
 <rectangle x1="22.86" y1="32.385" x2="49.53" y2="36.195" layer="22"/>
 <hole x="3.81" y="30.48" drill="3.2"/>
@@
 <attribute name="VALUE" x="32.639" y="15.367" size="0.8128" layer="21" font="vector" ratio="10" rot="R270"/>
 </element>
-<element name="LED1" library="SparkFun-LED" package="LED-0603" value="" x="48.895" y="25.4" smashed="yes" rot="R90">
-<attribute name="VALUE" x="50.546" y="27.305" size="1.27" layer="27" ratio="10" rot="R90"/>
-</element>
-<element name="R1" library="SparkFun-Passives" package="0805" value="330" x="45.085" y="25.4" smashed="yes" rot="R180">
-<attribute name="VALUE" x="43.688" y="26.924" size="1.016" layer="21" font="vector" ratio="15"/>
+<element name="LED1" library="SparkFun-LED" package="LED-0603" value="" x="29.21" y="25.4" smashed="yes" rot="R90">
+<attribute name="VALUE" x="30.861" y="27.305" size="1.27" layer="27" ratio="10" rot="R90"/>
+</element>
+<element name="R1" library="SparkFun-Passives" package="0805" value="330" x="25.4" y="25.4" smashed="yes" rot="R180">
+<attribute name="VALUE" x="24.003" y="26.924" size="1.016" layer="21" font="vector" ratio="15"/>
 </element>
 <element name="GPS0" library="OpenSpace" package="VENUS_GPS-NOSILK" value="VENUS_GPS-NOSILK" x="39.37" y="12.7" rot="MR90"/>
@@
 <attribute name="NAME" x="17.7038" y="1.1938" size="1.27" layer="25" ratio="10"/>
 </element>
+<element name="RX_EN" library="SparkFun-Passives" package="1X02" value="" x="45.72" y="25.4"/>
 </elements>
 <signals>
@@
 <wire x1="10.16" y1="7.62" x2="10.16" y2="17.78" width="0.254" layer="16"/>
 <wire x1="12.7" y1="7.62" x2="10.16" y2="7.62" width="0.254" layer="16"/>
-<wire x1="44.185" y1="25.4" x2="42.915" y2="24.13" width="0.254" layer="1"/>
-<wire x1="42.915" y1="24.13" x2="41.91" y2="24.13" width="0.254" layer="1"/>
-<wire x1="41.91" y1="24.13" x2="40.64" y2="22.86" width="0.254" layer="1"/>
 <wire x1="40.64" y1="22.86" x2="38.1" y2="25.4" width="0.254" layer="1"/>
 <wire x1="35.56" y1="18.045" x2="33.02" y2="18.045" width="0.254" layer="1"/>
@@
 <wire x1="41.91" y1="3.81" x2="31.75" y2="3.81" width="0.254" layer="16"/>
 <wire x1="31.75" y1="3.81" x2="30.48" y2="5.08" width="0.254" layer="16"/>
+<wire x1="24.5" y1="25.4" x2="22.86" y2="25.4" width="0.254" layer="1"/>
+<wire x1="22.86" y1="25.4" x2="21.59" y2="24.13" width="0.254" layer="1"/>
+<wire x1="21.59" y1="24.13" x2="21.59" y2="17.78" width="0.254" layer="1"/>
 </signal>
 <signal name="RX">
 <contactref element="ARDUINO" pad="RXI"/>
-<contactref element="LEVEL_SHIFT" pad="3"/>
-<wire x1="43.35" y1="14.59" x2="42.73" y2="13.97" width="0.254" layer="1"/>
-<wire x1="42.73" y1="13.97" x2="41.91" y2="13.97" width="0.254" layer="1"/>
-<via x="41.91" y="13.97" extent="1-16" drill="0.6"/>
-<wire x1="41.91" y1="13.97" x2="41.91" y2="16.51" width="0.254" layer="16"/>
-<wire x1="41.91" y1="16.51" x2="44.45" y2="19.05" width="0.254" layer="16"/>
-<wire x1="44.45" y1="19.05" x2="44.45" y2="21.59" width="0.254" layer="16"/>
-<wire x1="44.45" y1="21.59" x2="45.72" y2="22.86" width="0.254" layer="16"/>
+<contactref element="RX_EN" pad="1"/>
+<wire x1="45.72" y1="22.86" x2="45.72" y2="25.4" width="0.254" layer="16"/>
 </signal>
 <signal name="D4">
@@
 <contactref element="ARDUINO" pad="D4"/>
 <wire x1="33.02" y1="25.4" x2="33.02" y2="22.86" width="0.254" layer="16"/>
-<wire x1="33.02" y1="25.4" x2="34.29" y2="26.67" width="0.254" layer="1"/>
-<wire x1="34.29" y1="26.67" x2="48.26" y2="26.67" width="0.254" layer="1"/>
-<wire x1="48.26" y1="26.67" x2="49.53" y2="25.4" width="0.254" layer="1"/>
-<wire x1="49.53" y1="25.4" x2="49.645" y2="25.4" width="0.254" layer="1"/>
+<wire x1="29.96" y1="25.4" x2="33.02" y2="25.4" width="0.254" layer="1"/>
 </signal>
 <signal name="D3">
@@
 <contactref element="LED1" pad="C"/>
 <contactref element="R1" pad="1"/>
-<wire x1="48.145" y1="25.4" x2="45.985" y2="25.4" width="0.254" layer="1"/>
+<wire x1="26.3" y1="25.4" x2="28.46" y2="25.4" width="0.254" layer="1"/>
 </signal>
 <signal name="1.8V">
@@
 <wire x1="21.59" y1="6.35" x2="22.86" y2="7.62" width="0.254" layer="1"/>
 </signal>
+<signal name="N$7">
+<contactref element="LEVEL_SHIFT" pad="3"/>
+<contactref element="RX_EN" pad="2"/>
+<wire x1="48.26" y1="25.4" x2="49.53" y2="24.13" width="0.254" layer="16"/>
+<wire x1="49.53" y1="24.13" x2="49.53" y2="19.05" width="0.254" layer="16"/>
+<wire x1="49.53" y1="19.05" x2="48.26" y2="17.78" width="0.254" layer="16"/>
+<wire x1="48.26" y1="17.78" x2="43.18" y2="17.78" width="0.254" layer="16"/>
+<wire x1="43.18" y1="17.78" x2="41.91" y2="16.51" width="0.254" layer="16"/>
+<wire x1="41.91" y1="16.51" x2="41.91" y2="13.335" width="0.254" layer="16"/>
+<via x="41.91" y="13.335" extent="1-16" drill="0.6"/>
+<wire x1="41.91" y1="13.335" x2="43.165" y2="14.59" width="0.254" layer="1"/>
+<wire x1="43.165" y1="14.59" x2="43.35" y2="14.59" width="0.254" layer="1"/>
+</signal>
 </signals>
